File: inClassRobot.kicad_sch (KiCad schematic)
At the start: 53 parts, among them J1 BATT_CONN, J2 ENCODER_CONN, J3 Conn_01x04, J4 MT6701_CONN, J5 CONN_MPU6050, J6 M1_CONN, J7 M2_CONN, J8 ESP_CONN, J9 USB_C_Receptacle_USB2.0_14P, U1 LD1117S50TR_SOT223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

Commit message: Added docs
Connections:
- net +3.3V: no longer S2.1, S2.2, S2.3
- net +5V: now also S2.1
- net Vusb: now also S2.2
- new net +5V_REG: S2.3
Changed lines of the file:
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@@
 			)
 		)
-		(property "Value" "+3.3V"
-			(at 74.93 132.0799 90)
+		(property "Value" "Vusb"
+			(at 77.47 129.54 90)
 			(show_name no)
 			(do_not_autoplace no)
@@
 					(size 1.27 1.27)
 				)
-				(justify left)
 			)
 		)
@@
 			)
 		)
-		(property "Value" "+3.3V"
+		(property "Value" "+5V_REG"
 			(at 101.6 134.6199 90)
 			(show_name no)
@@
 			)
 		)
-		(property "Value" "+3.3V"
+		(property "Value" "+5V"
 			(at 101.6 129.5399 90)
 			(show_name no)
