File: inClassRobot.kicad_pcb (KiCad board)
At the start: 2 copper layers, 53 parts, among them J1 BATT_CONN, J2 ENCODER_CONN, J3 Conn_01x04, J4 MT6701_CONN, J5 CONN_MPU6050, J6 M1_CONN, J7 M2_CONN, J8 ESP_CONN, J9 USB_C_Receptacle_USB2.0_14P, U1 LD1117S50TR_SOT223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

Commit message: Added Board
Other:
- board outline added: 100 x 100 mm
Changed lines of the file:
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@@
 		)
+	)
+	(gr_rect
+		(start 116.5 56)
+		(end 216.5 156)
+		(stroke
+			(width 0.05)
+			(type solid)
+		)
+		(fill no)
+		(layer "Edge.Cuts")
 	)
 	(embedded_fonts no)
